Commit message: first commit after changes

File: ur_robot_server/urdf/ur_gripper.xacro (robot description, xacro)
@@ -26,5 +26,5 @@
   <xacro:include filename="$(find ur_robot_server)/urdf/ur_macro.xacro"/>
   <!-- include robotiq_85_gripper.urdf.xacro -->
-  <xacro:include filename="$(find robotiq_description)/urdf/robotiq_85_gripper.urdf.xacro"/>
+  <xacro:include filename="$(find ur_robot_server)/ur_robot_server/urdf/robotiq_85_gripper.xacro"/>
   <!--Declare arguments -->
   <xacro:arg name="joint_limit_params" default=""/>
@@ -71,9 +71,9 @@
   />
   <!-- include robot gripper -->
-  <xacro:robotiq_85_gripper prefix="" parent="tool0">
-    <origin xyz="0 0 0" rpy="0 -1.5707963 0"/>
+  <xacro:robotiq_85_gripper prefix="" parent="ee_link">
+    <origin xyz="0 0 0" rpy="0 0 0"/>
   </xacro:robotiq_85_gripper>
   <!--
-    Attach the Gazebo model to Gazebo's frame.
+    Attach the Gazebo model to Gazebo's world frame.
     Note: if you're looking to integrate a UR into a larger scene and need
     to add EEFs or other parts, DO NOT change this file or the 'world' link

File: ur_robot_server/urdf/ur_real.xacro (robot description, xacro)
@@ -25,6 +25,4 @@
   -->
   <xacro:include filename="$(find ur_robot_server)/urdf/ur_macro.xacro"/>
-  <!-- include robotiq_85_gripper.urdf.xacro -->
-  <xacro:include filename="$(find robotiq_description)/urdf/robotiq_85_gripper.urdf.xacro"/>
   <!--Declare arguments -->
   <xacro:arg name="joint_limit_params" default=""/>
@@ -70,10 +68,6 @@
     safety_k_position="$(arg safety_k_position)"
   />
-  <!-- include robot gripper -->
-  <xacro:robotiq_85_gripper prefix="" parent="tool0">
-    <origin xyz="0 0 0" rpy="0 -1.5707963 0"/>
-  </xacro:robotiq_85_gripper>
   <!--
-    Attach the Gazebo model to Gazebo's frame.
+    Attach the Gazebo model to Gazebo's world frame.
     Note: if you're looking to integrate a UR into a larger scene and need
     to add EEFs or other parts, DO NOT change this file or the 'world' link
@@ -98,22 +92,3 @@
     </joint>
   </xacro:if>
-  <!-- Grasp Plugin -->
-  <gazebo>
-      <plugin name="gazebo_grasp_fix" filename="libgazebo_grasp_fix.so">
-        <arm>
-          <arm_name>ur10e</arm_name>
-          <palm_link> gripper_finger1_inner_knuckle_link </palm_link>
-          <palm_link> gripper_finger2_inner_knuckle_link </palm_link>
-          <gripper_link> gripper_finger1_finger_tip_link </gripper_link>
-          <gripper_link> gripper_finger2_finger_tip_link </gripper_link>
-        </arm>
-        <forces_angle_tolerance>100</forces_angle_tolerance>
-        <update_rate>4</update_rate>
-        <grip_count_threshold>4</grip_count_threshold>
-        <max_grip_count>8</max_grip_count>
-        <release_tolerance>0.003</release_tolerance>
-        <disable_collisions_on_attach>false</disable_collisions_on_attach>
-        <contact_topic>__default_topic__</contact_topic>
-      </plugin>
-    </gazebo>
 </robot>
