Commit message: add realsense camera to robot

File: ur_robot_server/urdf/ur.xacro (robot description, xacro)
@@ -38,4 +38,10 @@
   <xacro:arg name="pitch" default="0.0"/>
   <xacro:arg name="yaw" default="0.0"/>
+  <!--xacro:arg name="x_camera" default="1.0"/>
+  <xacro:arg name="y_camera" default="1.0"/>
+  <xacro:arg name="z_camera" default="1.1"/>
+  <xacro:arg name="roll_camera" default="0.0"/>
+  <xacro:arg name="pitch_camera" default="0.0"/>
+  <xacro:arg name="yaw_camera" default="0.0"/-->
   <!--
     legal values:
@@ -87,6 +93,19 @@
     <origin xyz="$(arg x) $(arg y) $(arg z)" rpy="$(arg roll) $(arg pitch) $(arg yaw)" />
   </joint>
+  <xacro:if value="$(arg camera1_gazebo)">
+    <xacro:include filename="$(find realsense2_description)/urdf/_d435.urdf.xacro" />
+    <link name="camera_base_link" />
+    <xacro:sensor_d435 name="camera" topics_ns="camera" parent="camera_base_link" publish_pointcloud="false">
+      <origin xyz="0 0 0" rpy="0 0 0" />
+    </xacro:sensor_d435>
+    <joint name="camera_to_world_joint" type="fixed">
+      <parent link="world"/>
+      <child link="camera_base_link"/>
+      <origin xyz="$(arg camera1_link_x) $(arg camera1_link_y) $(arg camera1_link_z)"
+        rpy="$(arg camera1_link_roll) $(arg camera1_link_pitch) $(arg camera1_link_yaw)" />
+    </joint>
+  </xacro:if>
   <!-- simulated rgbd camera include -->
-  <xacro:if value="$(arg camera1_gazebo)">
+  <!--xacro:if value="$(arg camera1_gazebo)">
     <xacro:include filename="$(find scene_perception)/urdf/rgbd_camera_macro.xacro"/>
     <xacro:rgbd_camera_gazebo camera_name="camera1"/>
@@ -97,5 +116,5 @@
         rpy="$(arg camera1_link_roll) $(arg camera1_link_pitch) $(arg camera1_link_yaw)" />
     </joint>
-  </xacro:if>
+  </xacro:if-->
   <!-- Grasp Plugin -->
   <gazebo>

File: ur_robot_server/urdf/ur_gripper.xacro (robot description, xacro)
@@ -87,4 +87,14 @@
     <origin xyz="$(arg x) $(arg y) $(arg z)" rpy="$(arg roll) $(arg pitch) $(arg yaw)" />
   </joint>
+  <xacro:include filename="$(find realsense2_description)/urdf/_d435.urdf.xacro" />
+  <link name="camera_base_link" />
+  <xacro:sensor_d435 name="camera" topics_ns="camera" parent="camera_base_link" publish_pointcloud="true">
+    <origin xyz="0 0 0" rpy="0 0 0" />
+  </xacro:sensor_d435>
+  <joint name="world_camera_joint" type="fixed">
+    <parent link="world"/>
+    <child link="camera_base_link"/>
+    <origin xyz="0 0 0" rpy="$(arg roll) $(arg pitch) $(arg yaw)" />
+  </joint>
   <!-- simulated rgbd camera include -->
   <xacro:if value="$(arg camera1_gazebo)">
